File: Main/Recovery_DoubleStage.kicad_sch (KiCad schematic)
At the start: 54 parts, among them IC2 AP2210N-3.3TRG1, IC3 MMC5983MA, IC4 NEO-6M-0, IC5 BMP388, IC6 MPU-6050, J2 Conn_02x10_Counter_Clockwise, J3 Conn_Coaxial, J4 Conn_Coaxial, J5 MEM2075-00-140-01-A, J6 XT60PW-M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

Commit message: almost done with routing
Parts:
- removed TP7: MISO, TestPoint:TestPoint_Pad_D1.0mm, symbol Connector:TestPoint
- removed TP8: MOSI, TestPoint:TestPoint_Pad_D1.0mm, symbol Connector:TestPoint
- removed TP9: SCK, TestPoint:TestPoint_Pad_D1.0mm, symbol Connector:TestPoint
Connections:
- net ANT_NEO: now reaches IC4.11 (RF_IN), J3.1 (In), L1.2
- net ANT_LORA: now reaches J4.1 (In), U2.9 (ANT)
Changed lines of the file:
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@@
   (junction (at 242.57 159.385) (diameter 0) (color 0 0 0 0)
   )
+  (junction (at 83.947 138.684) (diameter 0) (color 0 0 0 0)
+  )
   (junction (at 37.719 37.719) (diameter 0) (color 0 0 0 0)
   )
@@
   (junction (at 21.971 42.672) (diameter 0) (color 0 0 0 0)
   )
+  (junction (at 244.348 50.165) (diameter 0) (color 0 0 0 0)
+  )
   (junction (at 237.49 151.765) (diameter 0) (color 0 0 0 0)
   )
@@
   (junction (at 36.83 117.856) (diameter 0) (color 0 0 0 0)
   )
+  (junction (at 98.552 156.591) (diameter 0) (color 0 0 0 0)
+  )
   (junction (at 36.83 92.71) (diameter 0) (color 0 0 0 0)
   )
@@
     (stroke (width 0) (type default) (color 0 0 0 0))
   )
-  (wire (pts (xy 167.132 17.907) (xy 168.148 17.907))
-    (stroke (width 0) (type default) (color 0 0 0 0))
-  )
   (wire (pts (xy 21.971 42.672) (xy 21.971 32.258))
     (stroke (width 0) (type default) (color 0 0 0 0))
@@
     (stroke (width 0) (type default) (color 0 0 0 0))
   )
-  (wire (pts (xy 167.132 19.812) (xy 167.132 19.685))
-    (stroke (width 0) (type default) (color 0 0 0 0))
-  )
   (wire (pts (xy 115.57 40.64) (xy 110.871 40.64))
     (stroke (width 0) (type default) (color 0 0 0 0))
@@
     (stroke (width 0) (type default) (color 0 0 0 0))
   )
+  (wire (pts (xy 98.552 156.591) (xy 99.06 156.591))
+    (stroke (width 0) (type default) (color 0 0 0 0))
+  )
   (wire (pts (xy 165.1 158.75) (xy 166.37 158.75))
     (stroke (width 0) (type default) (color 0 0 0 0))
@@
     (stroke (width 0) (type default) (color 0 0 0 0))
   )
+  (wire (pts (xy 98.552 156.591) (xy 98.552 157.48))
+    (stroke (width 0) (type default) (color 0 0 0 0))
+  )
   (wire (pts (xy 126.365 169.545) (xy 126.365 175.26))
     (stroke (width 0) (type default) (color 0 0 0 0))
@@
     (stroke (width 0) (type default) (color 0 0 0 0))
   )
-  (wire (pts (xy 167.132 19.685) (xy 169.418 19.685))
-    (stroke (width 0) (type default) (color 0 0 0 0))
-  )
   (wire (pts (xy 236.855 65.405) (xy 243.205 65.405))
     (stroke (width 0) (type default) (color 0 0 0 0))
@@
     (stroke (width 0) (type default) (color 0 0 0 0))
   )
+  (wire (pts (xy 244.348 50.165) (xy 245.11 50.165))
+    (stroke (width 0) (type default) (color 0 0 0 0))
+  )
   (wire (pts (xy 95.377 75.565) (xy 106.68 75.565))
     (stroke (width 0) (type default) (color 0 0 0 0))
@@
     (stroke (width 0) (type default) (color 0 0 0 0))
   )
+  (wire (pts (xy 244.348 50.165) (xy 244.348 55.753))
+    (stroke (width 0) (type default) (color 0 0 0 0))
+  )
   (wire (pts (xy 39.497 181.991) (xy 40.767 181.991))
     (stroke (width 0) (type default) (color 0 0 0 0))
@@
     (stroke (width 0) (type default) (color 0 0 0 0))
   )
-  (wire (pts (xy 95.377 156.591) (xy 99.06 156.591))
+  (wire (pts (xy 95.377 156.591) (xy 98.552 156.591))
     (stroke (width 0) (type default) (color 0 0 0 0))
   )
@@
     (stroke (width 0) (type default) (color 0 0 0 0))
   )
+  (wire (pts (xy 83.947 138.684) (xy 83.947 142.621))
+    (stroke (width 0) (type default) (color 0 0 0 0))
+  )
   (wire (pts (xy 90.17 88.9) (xy 85.09 88.9))
     (stroke (width 0) (type default) (color 0 0 0 0))
@@
     (stroke (width 0) (type default) (color 0 0 0 0))
   )
+  (wire (pts (xy 82.931 138.684) (xy 83.947 138.684))
+    (stroke (width 0) (type default) (color 0 0 0 0))
+  )
   (wire (pts (xy 230.505 158.369) (xy 233.299 158.369))
     (stroke (width 0) (type default) (color 0 0 0 0))
@@
     (stroke (width 0) (type default) (color 0 0 0 0))
   )
-  (wire (pts (xy 83.947 135.763) (xy 83.947 142.621))
+  (wire (pts (xy 83.947 135.763) (xy 83.947 138.684))
     (stroke (width 0) (type default) (color 0 0 0 0))
   )
@@
     (stroke (width 0) (type default) (color 0 0 0 0))
   )
-  (wire (pts (xy 167.132 21.717) (xy 170.434 21.717))
-    (stroke (width 0) (type default) (color 0 0 0 0))
-  )
   (wire (pts (xy 236.855 67.945) (xy 243.205 67.945))
     (stroke (width 0) (type default) (color 0 0 0 0))
@@
     (stroke (width 0) (type default) (color 0 0 0 0))
   )
-  (wire (pts (xy 236.855 50.165) (xy 245.11 50.165))
+  (wire (pts (xy 236.855 50.165) (xy 244.348 50.165))
     (stroke (width 0) (type default) (color 0 0 0 0))
   )
@@
     (effects (font (size 1.27 1.27)) (justify left bottom))
   )
+  (label "ANT_NEO" (at 98.552 157.48 270)
+    (effects (font (size 1.27 1.27)) (justify right bottom))
+  )
   (label "OPT1" (at 75.438 118.11 180)
     (effects (font (size 1.27 1.27)) (justify right bottom))
@@
     (effects (font (size 1.27 1.27)) (justify left bottom))
   )
-  (label "MISO" (at 167.132 17.907 180)
-    (effects (font (size 1.27 1.27)) (justify right bottom))
-  )
   (label "MPU_INT" (at 147.193 30.353 180)
     (effects (font (size 1.27 1.27)) (justify right bottom))
@@
     (effects (font (size 1.27 1.27)) (justify left bottom))
   )
-  (label "SCK" (at 167.132 21.717 180)
-    (effects (font (size 1.27 1.27)) (justify right bottom))
-  )
   (label "OPT4" (at 118.618 103.505 180)
     (effects (font (size 1.27 1.27)) (justify right bottom))
@@
     (effects (font (size 1.27 1.27)) (justify right bottom))
   )
+  (label "NEO_DECOUP" (at 82.931 138.684 180)
+    (effects (font (size 1.27 1.27)) (justify right bottom))
+  )
   (label "SD_CS" (at 146.939 35.941 180)
     (effects (font (size 1.27 1.27)) (justify right bottom))
@@
     (effects (font (size 1.27 1.27)) (justify right bottom))
   )
-  (label "MOSI" (at 167.132 19.812 180)
-    (effects (font (size 1.27 1.27)) (justify right bottom))
-  )
   (label "OPT5" (at 118.491 104.775 180)
     (effects (font (size 1.27 1.27)) (justify right bottom))
@@
     (effects (font (size 1.27 1.27)) (justify right bottom))
   )
+  (label "ANT_LORA" (at 244.348 53.213 180)
+    (effects (font (size 1.27 1.27)) (justify right bottom))
+  )
   (label "TX1" (at 39.243 175.768 180)
     (effects (font (size 1.27 1.27)) (justify right bottom))
@@
     (pin "1")
   )
-  (symbol (lib_id "Connector:TestPoint") (at 168.148 17.907 0) (unit 1)
-    (in_bom yes) (on_board yes)
-    (property "Reference" "TP7" (id 0) (at 168.656 12.954 0)
-      (effects (font (size 1.27 1.27)) (justify left))
-    )
-    (property "Value" "MISO" (id 1) (at 168.91 14.478 0)
-      (effects (font (size 1.27 1.27)) (justify left))
-    )
-    (property "Footprint" "TestPoint:TestPoint_Pad_D1.0mm" (id 2) (at 173.228 17.907 0)
-      (effects (font (size 1.27 1.27)) hide)
-    )
-    (property "Datasheet" "~" (id 3) (at 173.228 17.907 0)
-      (effects (font (size 1.27 1.27)) hide)
-    )
-    (pin "1")
-  )
-  (symbol (lib_id "Connector:TestPoint") (at 169.418 19.685 0) (unit 1)
-    (in_bom yes) (on_board yes)
-    (property "Reference" "TP8" (id 0) (at 170.434 15.7481 0)
-      (effects (font (size 1.27 1.27)) (justify left))
-    )
-    (property "Value" "MOSI" (id 1) (at 170.18 17.145 0)
-      (effects (font (size 1.27 1.27)) (justify left))
-    )
-    (property "Footprint" "TestPoint:TestPoint_Pad_D1.0mm" (id 2) (at 174.498 19.685 0)
-      (effects (font (size 1.27 1.27)) hide)
-    )
-    (property "Datasheet" "~" (id 3) (at 174.498 19.685 0)
-      (effects (font (size 1.27 1.27)) hide)
-    )
-    (pin "1")
-  )
   (symbol (lib_id "Switch:SW_Push") (at 114.3 86.741 0) (unit 1)
     (in_bom yes) (on_board yes)
@@
     (pin "2")
   )
-  (symbol (lib_id "Connector:TestPoint") (at 170.434 21.717 0) (unit 1)
-    (in_bom yes) (on_board yes)
-    (property "Reference" "TP9" (id 0) (at 171.196 18.542 0)
-      (effects (font (size 1.27 1.27)) (justify left))
-    )
-    (property "Value" "SCK" (id 1) (at 171.45 20.066 0)
-      (effects (font (size 1.27 1.27)) (justify left))
-    )
-    (property "Footprint" "TestPoint:TestPoint_Pad_D1.0mm" (id 2) (at 175.514 21.717 0)
-      (effects (font (size 1.27 1.27)) hide)
-    )
-    (property "Datasheet" "~" (id 3) (at 175.514 21.717 0)
-      (effects (font (size 1.27 1.27)) hide)
-    )
-    (pin "1")
-  )
   (symbol (lib_id "Device:C") (at 123.19 165.735 0) (unit 1)
     (in_bom yes) (on_board yes)
@@
       (reference "TP6") (unit 1) (value "LoRa_RESET") (footprint "TestPoint:TestPoint_Pad_D1.0mm")
     )
-    (path "/1764af04-4b30-44cb-9d80-b096de98a266"
-      (reference "TP7") (unit 1) (value "MISO") (footprint "TestPoint:TestPoint_Pad_D1.0mm")
-    )
-    (path "/18109353-3125-4335-900f-bdc4aee093cb"
-      (reference "TP8") (unit 1) (value "MOSI") (footprint "TestPoint:TestPoint_Pad_D1.0mm")
-    )
-    (path "/4b93eb82-e5a3-4aac-905e-2d5c4910c98f"
-      (reference "TP9") (unit 1) (value "SCK") (footprint "TestPoint:TestPoint_Pad_D1.0mm")
-    )
     (path "/df36cb6e-e4fe-4646-a522-5f4686f4ab13"
