File: Main/Recovery_DoubleStage.kicad_sch (KiCad schematic)
At the start: 55 parts, among them IC2 AP2210N-3.3TRG1, IC3 MMC5983MA, IC4 NEO-6M-0, IC5 BMP388, IC6 MPU-6050, J2 Conn_02x10_Counter_Clockwise, J3 Conn_Coaxial, J4 Conn_Coaxial, J5 MEM2075-00-140-01-A, J6 JSTXH-1x02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

Commit message: added relative paths
Parts:
- removed C17, C18: 10u, Capacitor_SMD:C_0603_1608Metric, symbol Device:C
- removed U1: NCP5501DT50RKG, Footprint:NCP5501DT50RKG, symbol custom:NCP5501DT50RKG
- H1, H2, H3, H4: footprint MountingHole:MountingHole_2.1mm -> MountingHole:MountingHole_3.2mm_M3
Connections:
- net ID1: no longer J2.19 (Pin_19)
- net ID2: no longer J2.18 (Pin_18)
- net ID3: no longer J2.15 (Pin_15)
- net IGNITION: no longer J2.14 (Pin_14)
- net Relay_1: no longer J2.17 (Pin_17)
- net Relay_2: no longer J2.16 (Pin_16)
Other:
- added sheet igniter (igniter.kicad_sch)

Commit message: reviewed design. starting routing
Parts:
- removed C19, C20: 10u, Capacitor_SMD:C_0603_1608Metric, symbol Device:C
- removed IC2: AP2210N-3.3TRG1, Footprint:SOT95P280X145-3N, symbol AP2210N-3.3TRG1:AP2210N-3.3TRG1
- removed SW1: SW_Push, Footprint:PTS815SJK250SMTRLFS, symbol Switch:SW_Push
- added C17: 4.7u, Capacitor_SMD:C_0603_1608Metric, symbol Device:C
- added C18: 10u, Capacitor_SMD:C_0603_1608Metric, symbol Device:C
- added L2: 1uH, Inductor_SMD:L_0805_2012Metric, symbol Device:L
- added R25: 100k, Resistor_SMD:R_0603_1608Metric, symbol Device:R
- added TP7: TestPoint, TestPoint:TestPoint_Pad_D1.0mm, symbol Connector:TestPoint
- added U3: ADP2108AUJ-3.3, Package_TO_SOT_SMD:TSOT-23-5, symbol Regulator_Switching:ADP2108AUJ-3.3
Connections:
- net +3V3: now also C18.2, L2.2, R25.2, U3.4 (FB)
- net +BATT: now also C17.2, U3.1 (Vin), U3.3 (EN)
- net GND: now also C17.1, C18.1, U3.2 (GND)
- net LoRa_CS: now also R25.1
- net LoRa_Ready: now reaches U2.14 (DIO0)
- net LoRa_Ready: now also TP7.1
- net ANT_LORA: no longer names the net of J4.1 (In), U2.9 (ANT)
- new net: L2.1, U3.5 (SW)
- no-connect marks 41 -> 40
Other:
- sheet microcontroller ports: added LoRa_Ready; removed none

Commit message: finalized pcb
Parts:
- removed R9: 10k, Resistor_SMD:R_0603_1608Metric, symbol Device:R
- removed TP12: SDA, TestPoint:TestPoint_Pad_D1.0mm, symbol Connector:TestPoint
- removed TP13: SCL, TestPoint:TestPoint_Pad_D1.0mm, symbol Connector:TestPoint
Connections:
- net +3V3: now also BZ1.2 (+), D2.3 (K); no longer C14.2, C15.2, L1.1
- net +5V: no longer BZ1.2 (+), D2.3 (K)
- net MISO: now also J2.16 (Pin_16)
- net MOSI: now also J2.15 (Pin_15)
- net SCK: now also J2.14 (Pin_14)
- net SD_CS: now also J5.P2 (CD/DAT3); no longer J5.P9 (CD)
- net at IC4.8 (RESERVED_2), IC4.9 (VCC_RF): now also C14.2, C15.2, L1.1
- new net SD_CD: J5.P9 (CD)
Other:
- sheet microcontroller ports: added SD_CD, igniter1, igniter2, igniter3; removed IGNITION
- moved on the sheet: C14, C15, L1
