File: Main/igniter.kicad_sch (KiCad schematic)
At the start: 28 parts, among them IC7 PS2801C-4-F3-A, J10 Screw_Terminal_01x02, J7 Screw_Terminal_01x06, Q2 BSS138, Q3 BSS138, Q4 BSS138, U1 Opamp_Quad

Commit message: added relative paths
Changed lines of the file:
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@@
   )
   (symbol (lib_id "power:GND1") (at 86.995 73.406 0) (mirror y) (unit 1)
-    (in_bom yes) (on_board yes) (fields_autoplaced)
-    (property "Reference" "#PWR?" (id 0) (at 86.995 79.756 0)
+    (in_bom yes) (on_board yes)
+    (property "Reference" "#PWR0111" (id 0) (at 86.995 79.756 0)
       (effects (font (size 1.27 1.27)) hide)
     )
-    (property "Value" "GND1" (id 1) (at 86.995 78.486 0))
+    (property "Value" "GND1" (id 1) (at 83.185 74.422 0))
     (property "Footprint" "" (id 2) (at 86.995 73.406 0)
       (effects (font (size 1.27 1.27)) hide)

Commit message: reviewed design. starting routing
Parts:
- removed J10: Screw_Terminal_01x02, symbol Connector:Screw_Terminal_01x02
- added J8: JSTXH-1x02, Connector_JST:JST_XH_B2B-XH-AM_1x02_P2.50mm_Vertical, symbol XT60PW-M:XT60PW-M
Connections:
- net +9V: now also J8.1 (+)
- net GND1: now also J8.2 (-)
Changed lines of the file:
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@@
     (stroke (width 0) (type default) (color 0 0 0 0))
   )
-  (wire (pts (xy 32.766 45.085) (xy 32.766 46.482))
+  (wire (pts (xy 25.908 45.593) (xy 25.908 46.99))
     (stroke (width 0) (type default) (color 0 0 0 0))
   )
@@
     (stroke (width 0) (type default) (color 0 0 0 0))
   )
-  (wire (pts (xy 31.369 49.022) (xy 33.02 49.022))
+  (wire (pts (xy 27.305 49.53) (xy 25.654 49.53))
     (stroke (width 0) (type default) (color 0 0 0 0))
   )
@@
     (stroke (width 0) (type default) (color 0 0 0 0))
   )
-  (wire (pts (xy 119.507 62.992) (xy 119.507 62.103))
-    (stroke (width 0) (type default) (color 0 0 0 0))
-  )
   (wire (pts (xy 69.469 121.158) (xy 72.009 121.158))
     (stroke (width 0) (type default) (color 0 0 0 0))
@@
     (stroke (width 0) (type default) (color 0 0 0 0))
   )
-  (wire (pts (xy 119.507 62.103) (xy 120.269 62.103))
-    (stroke (width 0) (type default) (color 0 0 0 0))
-  )
   (wire (pts (xy 201.041 92.329) (xy 203.581 92.329))
     (stroke (width 0) (type default) (color 0 0 0 0))
@@
     (stroke (width 0) (type default) (color 0 0 0 0))
   )
-  (wire (pts (xy 33.02 49.022) (xy 33.02 50.165))
+  (wire (pts (xy 25.654 49.53) (xy 25.654 50.673))
     (stroke (width 0) (type default) (color 0 0 0 0))
   )
@@
     (stroke (width 0) (type default) (color 0 0 0 0))
   )
-  (wire (pts (xy 32.766 46.482) (xy 31.369 46.482))
+  (wire (pts (xy 25.908 46.99) (xy 27.305 46.99))
     (stroke (width 0) (type default) (color 0 0 0 0))
   )
@@
     (pin "1")
   )
-  (symbol (lib_id "power:GND1") (at 119.507 62.992 0) (mirror y) (unit 1)
-    (in_bom yes) (on_board yes) (fields_autoplaced)
-    (property "Reference" "#PWR056" (id 0) (at 119.507 69.342 0)
-      (effects (font (size 1.27 1.27)) hide)
-    )
-    (property "Value" "GND1" (id 1) (at 119.507 68.072 0))
-    (property "Footprint" "" (id 2) (at 119.507 62.992 0)
-      (effects (font (size 1.27 1.27)) hide)
-    )
-    (property "Datasheet" "" (id 3) (at 119.507 62.992 0)
-      (effects (font (size 1.27 1.27)) hide)
-    )
-    (pin "1")
-  )
   (symbol (lib_id "G6RL-1-DC3:G6RL-1-DC3") (at 68.326 54.991 0) (unit 1)
     (in_bom yes) (on_board yes)
@@
     (pin "1")
   )
+  (symbol (lib_id "XT60PW-M:XT60PW-M") (at 37.465 49.53 0) (unit 1)
+    (in_bom yes) (on_board yes) (fields_autoplaced)
+    (property "Reference" "J8" (id 0) (at 43.307 46.9899 0)
+      (effects (font (size 1.27 1.27)) (justify left))
+    )
+    (property "Value" "JSTXH-1x02" (id 1) (at 43.307 49.5299 0)
+      (effects (font (size 1.27 1.27)) (justify left))
+    )
+    (property "Footprint" "Connector_JST:JST_XH_B2B-XH-AM_1x02_P2.50mm_Vertical" (id 2) (at 37.465 49.53 0)
+      (effects (font (size 1.27 1.27)) (justify bottom) hide)
+    )
+    (property "Datasheet" "" (id 3) (at 37.465 49.53 0)
+      (effects (font (size 1.27 1.27)) hide)
+    )
+    (property "STANDARD" "Manufacturer recommendations" (id 4) (at 37.465 49.53 0)
+      (effects (font (size 1.27 1.27)) (justify bottom) hide)
+    )
+    (property "MAXIMUM_PACKAGE_HEIGHT" "8.4 mm" (id 5) (at 37.465 49.53 0)
+      (effects (font (size 1.27 1.27)) (justify bottom) hide)
+    )
+    (property "MANUFACTURER" "AMASS" (id 6) (at 37.465 49.53 0)
+      (effects (font (size 1.27 1.27)) (justify bottom) hide)
+    )
+    (property "PARTREV" "V1.2" (id 7) (at 37.465 49.53 0)
+      (effects (font (size 1.27 1.27)) (justify bottom) hide)
+    )
+    (pin "1")
+    (pin "2")
+  )
   (symbol (lib_id "power:+9V") (at 70.866 113.411 0) (unit 1)
     (in_bom yes) (on_board yes)
@@
     (pin "1")
   )
-  (symbol (lib_id "Connector:Screw_Terminal_01x02") (at 26.289 46.482 0) (mirror y) (unit 1)
-    (in_bom yes) (on_board yes)
-    (property "Reference" "J10" (id 0) (at 26.289 39.37 0))
-    (property "Value" "Screw_Terminal_01x02" (id 1) (at 24.384 41.021 0))
-    (property "Footprint" "" (id 2) (at 26.289 46.482 0)
-      (effects (font (size 1.27 1.27)) hide)
-    )
-    (property "Datasheet" "~" (id 3) (at 26.289 46.482 0)
-      (effects (font (size 1.27 1.27)) hide)
-    )
-    (pin "1")
-    (pin "2")
-  )
   (symbol (lib_id "power:GND") (at 156.718 26.162 0) (unit 1)
     (in_bom yes) (on_board yes)
@@
     (pin "1")
   )
-  (symbol (lib_id "power:GND1") (at 33.02 50.165 0) (mirror y) (unit 1)
-    (in_bom yes) (on_board yes) (fields_autoplaced)
-    (property "Reference" "#PWR072" (id 0) (at 33.02 56.515 0)
-      (effects (font (size 1.27 1.27)) hide)
-    )
-    (property "Value" "GND1" (id 1) (at 33.02 55.245 0))
-    (property "Footprint" "" (id 2) (at 33.02 50.165 0)
-      (effects (font (size 1.27 1.27)) hide)
-    )
-    (property "Datasheet" "" (id 3) (at 33.02 50.165 0)
+  (symbol (lib_id "power:GND1") (at 25.654 50.673 0) (unit 1)
+    (in_bom yes) (on_board yes) (fields_autoplaced)
+    (property "Reference" "#PWR072" (id 0) (at 25.654 57.023 0)
+      (effects (font (size 1.27 1.27)) hide)
+    )
+    (property "Value" "GND1" (id 1) (at 25.654 55.753 0))
+    (property "Footprint" "" (id 2) (at 25.654 50.673 0)
+      (effects (font (size 1.27 1.27)) hide)
+    )
+    (property "Datasheet" "" (id 3) (at 25.654 50.673 0)
       (effects (font (size 1.27 1.27)) hide)
     )
@@
     (pin "4")
   )
-  (symbol (lib_id "power:+9V") (at 32.766 45.085 0) (unit 1)
-    (in_bom yes) (on_board yes)
-    (property "Reference" "#PWR071" (id 0) (at 32.766 48.895 0)
-      (effects (font (size 1.27 1.27)) hide)
-    )
-    (property "Value" "+9V" (id 1) (at 36.068 44.704 0))
-    (property "Footprint" "" (id 2) (at 32.766 45.085 0)
-      (effects (font (size 1.27 1.27)) hide)
-    )
-    (property "Datasheet" "" (id 3) (at 32.766 45.085 0)
-      (effects (font (size 1.27 1.27)) hide)
-    )
+  (symbol (lib_id "power:+9V") (at 25.908 45.593 0) (mirror y) (unit 1)
+    (in_bom yes) (on_board yes)
+    (property "Reference" "#PWR071" (id 0) (at 25.908 49.403 0)
+      (effects (font (size 1.27 1.27)) hide)
+    )
+    (property "Value" "+9V" (id 1) (at 22.606 45.212 0))
+    (property "Footprint" "" (id 2) (at 25.908 45.593 0)
+      (effects (font (size 1.27 1.27)) hide)
+    )
+    (property "Datasheet" "" (id 3) (at 25.908 45.593 0)
+      (effects (font (size 1.27 1.27)) hide)
+    )

Commit message: finalized pcb
Parts:
- removed U1: Opamp_Quad, Attiny414:SOIC127P600X175-14N, symbol Device:Opamp_Quad
- added C19: C_Polarized, Capacitor_SMD:CP_Elec_6.3x7.7, symbol Device:C_Polarized
- added R29, R30, R31: 100k, Resistor_SMD:R_0603_1608Metric, symbol Device:R
- added R32: 100, Resistor_SMD:R_0603_1608Metric, symbol Device:R
- added U1: LM339, Package_SO:TSSOP-14_4.4x5mm_P0.65mm, symbol Comparator:LM339
- R13: value 1k -> 100k
- R5: value 100k -> 1k
Connections:
- net +3V3: now also C19.1
- net +9V: now also R13.1, R29.1, R30.1, R31.1, R32.2, U1.3 (V+); no longer O1.4 (NC), O2.4 (NC), O3.4 (NC), R5.1
- net GND: now also R16.1, R18.1, R23.1, C19.2
- net GND1: now also R5.2, U1.12 (V-); no longer IC7.2 (CATHODE_1), IC7.4 (CATHODE_2), IC7.6 (CATHODE_3), R13.2
- net osense1_hv: now also IC7.2 (CATHODE_1), U1.2; no longer IC7.1 (ANODE_1)
- net osense2_hv: now also IC7.4 (CATHODE_2), U1.1; no longer IC7.3 (ANODE_2)
- net osense3_hv: now also IC7.6 (CATHODE_3), U1.13; no longer IC7.5 (ANODE_3)
- net at Q2.1 (G), R15.2: now also R16.2; no longer R16.1
- net at D3.2 (A), O1.5 (COIL_2), Q2.3 (D): no longer R16.2
- net at Q3.1 (G), R17.2: now also R18.2; no longer R18.1
- net at D5.2 (A), O3.5 (COIL_2), Q4.3 (D): no longer R23.2
- net at Q4.1 (G), R21.2: now also R23.2; no longer R23.1
- net at R12.1: now also R13.2, U1.5 (+); no longer R5.2
- net at D4.2 (A), O2.5 (COIL_2), Q3.3 (D): no longer R18.2
- net at R14.1: now also R29.2, U1.7 (+); no longer R11.2
- net at R10.2: now also R5.1, U1.11 (+); no longer R13.1
- new net: IC7.1 (ANODE_1), IC7.3 (ANODE_2), IC7.5 (ANODE_3), R32.1
- new net sense_1: O1.4 (NC), R30.2, U1.4 (-)
- new net sense_2: O2.4 (NC), R31.2, U1.6 (-)
- new net sense_3: O3.4 (NC), R11.2, U1.10 (-)
Other:
- moved on the sheet: R16, R18, R23
