File: Main/microcontroller.kicad_sch (KiCad schematic)
At the start: 13 parts, among them IC1 ATMEGA2560-16AU, J1 ICSP, Y1 CSTNE16M0V530000R0

Commit message: almost done with routing
Connections:
- net ID1: now also IC1.55 (PC2_(A10)); no longer IC1.57 (PC4_(A12))
- net ID2: now also IC1.56 (PC3_(A11)); no longer IC1.58 (PC5_(A13))
- net ID3: now also IC1.57 (PC4_(A12)); no longer IC1.55 (PC2_(A10))
- net IGNITION: now also IC1.58 (PC5_(A13)); no longer IC1.56 (PC3_(A11))

Commit message: reviewed design. starting routing
Parts:
- added R24: 330k, Resistor_SMD:R_0603_1608Metric, symbol Device:R
- added R26, R27, R28: 330, Resistor_SMD:R_0603_1608Metric, symbol Device:R
- added SW1: SW_Push, Footprint:PTS815SJK250SMTRLFS, symbol Switch:SW_Push
- C1: value 22p -> 100nF
Connections:
- net GND: now also SW1.1
- net MISO: now also R26.1, R26.2
- net MOSI: now also R27.1, R27.2
- net RESET: now also R24.2
- net SCK: now also R28.1, R28.2
- net LoRa_Ready: now reaches IC1.76 (PA2_(AD2))
- new net: R24.1, SW1.2
- no-connect marks 59 -> 58
Changed lines of the file:
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@@
   (no_connect (at 142.24 118.11))
   (no_connect (at 142.24 198.12))
-  (no_connect (at 142.24 59.69))
   (no_connect (at 71.12 207.01))
   (no_connect (at 142.24 49.53))
@@
     (stroke (width 0) (type default) (color 0 0 0 0))
   )
+  (wire (pts (xy 46.482 26.67) (xy 46.482 17.526))
+    (stroke (width 0) (type default) (color 0 0 0 0))
+  )
   (wire (pts (xy 66.929 33.02) (xy 116.84 33.02))
     (stroke (width 0) (type default) (color 0 0 0 0))
@@
     (stroke (width 0) (type default) (color 0 0 0 0))
   )
-  (wire (pts (xy 161.163 92.71) (xy 168.148 92.71))
+  (wire (pts (xy 161.163 92.71) (xy 171.45 92.71))
     (stroke (width 0) (type default) (color 0 0 0 0))
   )
@@
     (stroke (width 0) (type default) (color 0 0 0 0))
   )
+  (wire (pts (xy 179.07 92.71) (xy 185.42 92.71))
+    (stroke (width 0) (type default) (color 0 0 0 0))
+  )
   (wire (pts (xy 142.24 77.47) (xy 144.272 77.47))
     (stroke (width 0) (type default) (color 0 0 0 0))
   )
-  (wire (pts (xy 164.338 90.17) (xy 168.148 90.17))
+  (wire (pts (xy 164.338 90.17) (xy 171.45 90.17))
     (stroke (width 0) (type default) (color 0 0 0 0))
   )
@@
     (stroke (width 0) (type default) (color 0 0 0 0))
   )
+  (wire (pts (xy 65.659 26.67) (xy 66.929 26.67))
+    (stroke (width 0) (type default) (color 0 0 0 0))
+  )
   (wire (pts (xy 196.85 55.88) (xy 196.85 54.61))
     (stroke (width 0) (type default) (color 0 0 0 0))
   )
+  (wire (pts (xy 56.642 26.67) (xy 58.039 26.67))
+    (stroke (width 0) (type default) (color 0 0 0 0))
+  )
   (wire (pts (xy 233.045 62.23) (xy 233.045 65.405))
     (stroke (width 0) (type default) (color 0 0 0 0))
@@
     (stroke (width 0) (type default) (color 0 0 0 0))
   )
+  (wire (pts (xy 44.323 17.526) (xy 46.482 17.526))
+    (stroke (width 0) (type default) (color 0 0 0 0))
+  )
   (wire (pts (xy 142.24 139.7) (xy 146.05 139.7))
     (stroke (width 0) (type default) (color 0 0 0 0))
@@
     (stroke (width 0) (type default) (color 0 0 0 0))
   )
+  (wire (pts (xy 142.24 59.69) (xy 145.923 59.69))
+    (stroke (width 0) (type default) (color 0 0 0 0))
+  )
   (wire (pts (xy 142.24 113.03) (xy 145.796 113.03))
     (stroke (width 0) (type default) (color 0 0 0 0))
@@
     (stroke (width 0) (type default) (color 0 0 0 0))
   )
+  (wire (pts (xy 179.07 90.17) (xy 185.42 90.17))
+    (stroke (width 0) (type default) (color 0 0 0 0))
+  )
   (wire (pts (xy 161.163 85.09) (xy 161.163 92.71))
     (stroke (width 0) (type default) (color 0 0 0 0))
@@
     (stroke (width 0) (type default) (color 0 0 0 0))
   )
-  (wire (pts (xy 167.513 87.63) (xy 168.148 87.63))
+  (wire (pts (xy 167.513 87.63) (xy 171.45 87.63))
     (stroke (width 0) (type default) (color 0 0 0 0))
   )
@@
     (stroke (width 0) (type default) (color 0 0 0 0))
   )
+  (wire (pts (xy 179.07 87.63) (xy 185.42 87.63))
+    (stroke (width 0) (type default) (color 0 0 0 0))
+  )
   (wire (pts (xy 64.516 33.02) (xy 66.929 33.02))
     (stroke (width 0) (type default) (color 0 0 0 0))
@@
   )
   (wire (pts (xy 71.12 95.25) (xy 68.58 95.25))
+    (stroke (width 0) (type default) (color 0 0 0 0))
+  )
+  (wire (pts (xy 66.929 26.67) (xy 66.929 33.02))
     (stroke (width 0) (type default) (color 0 0 0 0))
   )
@@
     (effects (font (size 1.27 1.27)) (justify left bottom))
   )
-  (label "SCK" (at 168.148 92.71 0)
-    (effects (font (size 1.27 1.27)) (justify left bottom))
-  )
   (label "SCK" (at 177.8 59.055 180)
     (effects (font (size 1.27 1.27)) (justify right bottom))
   )
+  (label "MISO" (at 167.513 85.09 90)
+    (effects (font (size 1.27 1.27)) (justify left bottom))
+  )
   (label "MOSI" (at 198.755 58.42 0)
     (effects (font (size 1.27 1.27)) (justify left bottom))
@@
     (effects (font (size 1.27 1.27)) (justify right bottom))
   )
-  (label "MOSI" (at 168.148 90.17 0)
+  (label "MOSI" (at 164.338 85.09 90)
     (effects (font (size 1.27 1.27)) (justify left bottom))
   )
-  (label "MISO" (at 168.148 87.63 0)
+  (label "SCK" (at 161.163 85.09 90)
     (effects (font (size 1.27 1.27)) (justify left bottom))
   )
@@
     (effects (font (size 1.27 1.27)) (justify left))
   )
+  (hierarchical_label "LoRa_Ready" (shape input) (at 145.923 59.69 0)
+    (effects (font (size 1.27 1.27)) (justify left))
+  )
+  (hierarchical_label "SCK" (shape input) (at 185.42 92.71 0)
+    (effects (font (size 1.27 1.27)) (justify left))
+  )
   (hierarchical_label "LoRa_RESET" (shape input) (at 145.923 64.77 0)
     (effects (font (size 1.27 1.27)) (justify left))
@@
     (effects (font (size 1.27 1.27)) (justify left))
   )
+  (hierarchical_label "MISO" (shape input) (at 185.42 87.63 0)
+    (effects (font (size 1.27 1.27)) (justify left))
+  )
   (hierarchical_label "SD_CS" (shape input) (at 144.399 95.25 0)
     (effects (font (size 1.27 1.27)) (justify left))
@@
     (effects (font (size 1.27 1.27)) (justify left))
   )
-  (hierarchical_label "SCK" (shape input) (at 161.163 85.09 90)
+  (hierarchical_label "MOSI" (shape input) (at 185.42 90.17 0)
     (effects (font (size 1.27 1.27)) (justify left))
   )
@@
     (effects (font (size 1.27 1.27)) (justify left))
   )
-  (hierarchical_label "MISO" (shape input) (at 167.513 85.09 90)
-    (effects (font (size 1.27 1.27)) (justify left))
-  )
-  (hierarchical_label "MOSI" (shape input) (at 164.338 85.09 90)
-    (effects (font (size 1.27 1.27)) (justify left))
-  )
   (hierarchical_label "OPT1" (shape input) (at 144.272 77.47 0)
     (effects (font (size 1.27 1.27)) (justify left))
@@
     (pin "2")
   )
+  (symbol (lib_id "Device:R") (at 61.849 26.67 90) (unit 1)
+    (in_bom yes) (on_board yes) (fields_autoplaced)
+    (property "Reference" "R24" (id 0) (at 61.849 20.32 90))
+    (property "Value" "330k" (id 1) (at 61.849 22.86 90))
+    (property "Footprint" "Resistor_SMD:R_0603_1608Metric" (id 2) (at 61.849 28.448 90)
+      (effects (font (size 1.27 1.27)) hide)
+    )
+    (property "Datasheet" "~" (id 3) (at 61.849 26.67 0)
+      (effects (font (size 1.27 1.27)) hide)
+    )
+    (pin "1")
+    (pin "2")
+  )
   (symbol (lib_id "Device:C") (at 120.65 40.64 90) (unit 1)
     (in_bom yes) (on_board yes) (fields_autoplaced)
     (property "Reference" "C1" (id 0) (at 120.65 33.02 90))
-    (property "Value" "22p" (id 1) (at 120.65 35.56 90))
+    (property "Value" "100nF" (id 1) (at 120.65 35.56 90))
     (property "Footprint" "Capacitor_SMD:C_0603_1608Metric" (id 2) (at 124.46 39.6748 0)
       (effects (font (size 1.27 1.27)) hide)
     )
     (property "Datasheet" "~" (id 3) (at 120.65 40.64 0)
+      (effects (font (size 1.27 1.27)) hide)
+    )
+    (pin "1")
+    (pin "2")
+  )
+  (symbol (lib_id "Switch:SW_Push") (at 51.562 26.67 0) (unit 1)
+    (in_bom yes) (on_board yes)
+    (property "Reference" "SW1" (id 0) (at 52.197 28.829 0))
+    (property "Value" "SW_Push" (id 1) (at 45.72 28.829 0))
+    (property "Footprint" "Footprint:PTS815SJK250SMTRLFS" (id 2) (at 51.562 21.59 0)
+      (effects (font (size 1.27 1.27)) hide)
+    )
+    (property "Datasheet" "~" (id 3) (at 51.562 21.59 0)
       (effects (font (size 1.27 1.27)) hide)
     )
@@
     )
     (property "Datasheet" "" (id 3) (at 116.84 19.05 0)
+      (effects (font (size 1.27 1.27)) hide)
+    )
+    (pin "1")
+  )
+  (symbol (lib_id "power:GND") (at 44.323 17.526 0) (unit 1)
+    (in_bom yes) (on_board yes)
+    (property "Reference" "#PWR0112" (id 0) (at 44.323 23.876 0)
+      (effects (font (size 1.27 1.27)) hide)
+    )
+    (property "Value" "GND" (id 1) (at 44.323 21.082 0))
+    (property "Footprint" "" (id 2) (at 44.323 17.526 0)
+      (effects (font (size 1.27 1.27)) hide)
+    )
+    (property "Datasheet" "" (id 3) (at 44.323 17.526 0)
       (effects (font (size 1.27 1.27)) hide)
     )
@@
     (pin "99")
   )
+  (symbol (lib_id "Device:R") (at 175.26 87.63 90) (unit 1)
+    (in_bom yes) (on_board yes)
+    (property "Reference" "R26" (id 0) (at 181.356 87.884 90))
+    (property "Value" "330" (id 1) (at 175.006 87.757 90))
+    (property "Footprint" "Resistor_SMD:R_0603_1608Metric" (id 2) (at 175.26 89.408 90)
+      (effects (font (size 1.27 1.27)) hide)
+    )
+    (property "Datasheet" "~" (id 3) (at 175.26 87.63 0)
+      (effects (font (size 1.27 1.27)) hide)
+    )
+    (pin "1")
+    (pin "2")
+  )
+  (symbol (lib_id "Device:R") (at 175.26 90.17 90) (unit 1)
+    (in_bom yes) (on_board yes)
+    (property "Reference" "R27" (id 0) (at 181.356 90.17 90))
+    (property "Value" "330" (id 1) (at 175.006 90.17 90))
+    (property "Footprint" "Resistor_SMD:R_0603_1608Metric" (id 2) (at 175.26 91.948 90)
+      (effects (font (size 1.27 1.27)) hide)
+    )
+    (property "Datasheet" "~" (id 3) (at 175.26 90.17 0)
+      (effects (font (size 1.27 1.27)) hide)
+    )
+    (pin "1")
+    (pin "2")
+  )
   (symbol (lib_id "power:+3V3") (at 196.85 54.61 0) (unit 1)
     (in_bom yes) (on_board yes) (fields_autoplaced)
@@
     (pin "1")
   )
+  (symbol (lib_id "Device:R") (at 175.26 92.71 90) (unit 1)
+    (in_bom yes) (on_board yes)
+    (property "Reference" "R28" (id 0) (at 181.229 92.837 90))
+    (property "Value" "330" (id 1) (at 175.133 92.583 90))
+    (property "Footprint" "Resistor_SMD:R_0603_1608Metric" (id 2) (at 175.26 94.488 90)
+      (effects (font (size 1.27 1.27)) hide)
+    )
+    (property "Datasheet" "~" (id 3) (at 175.26 92.71 0)
+      (effects (font (size 1.27 1.27)) hide)
+    )
+    (pin "1")
+    (pin "2")
+  )
   (symbol (lib_id "power:+3V3") (at 34.29 69.85 90) (unit 1)

Commit message: finalized pcb
Connections:
- net MISO: no longer IC1.22 ((MISO/PCINT3)_PB3), J1.1 (Pin_1), R26.1
- net MOSI: no longer IC1.21 ((MOSI/PCINT2)_PB2), J1.4 (Pin_4), R27.1
- net SCK: no longer IC1.20 ((SCK/PCINT1)_PB1), J1.3 (Pin_3), R28.1
- net SD_CD: now reaches IC1.6 ((OC3B/INT4)_PE4)
- net IGNITION renamed igniter1
- net Relay_1 renamed igniter2
- net Relay_2 renamed igniter3
- new net MISO_JTAG: IC1.22 ((MISO/PCINT3)_PB3), J1.1 (Pin_1), R26.1
- new net MOSI_JTAG: IC1.21 ((MOSI/PCINT2)_PB2), J1.4 (Pin_4), R27.1
- new net SCK_JTAG: IC1.20 ((SCK/PCINT1)_PB1), J1.3 (Pin_3), R28.1
- no-connect marks 58 -> 57
Changed lines of the file:
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@@
   (no_connect (at 142.24 127))
   (no_connect (at 71.12 124.46))
-  (no_connect (at 142.24 153.67))
   (no_connect (at 142.24 115.57))
   (no_connect (at 142.24 182.88))
@@
     (stroke (width 0) (type default) (color 0 0 0 0))
   )
+  (wire (pts (xy 142.24 153.67) (xy 143.637 153.67))
+    (stroke (width 0) (type default) (color 0 0 0 0))
+  )
   (wire (pts (xy 64.389 63.5) (xy 71.12 63.5))
     (stroke (width 0) (type default) (color 0 0 0 0))
@@
     (effects (font (size 1.27 1.27)) (justify left bottom))
   )
-  (label "SCK" (at 177.8 59.055 180)
+  (label "SCK_JTAG" (at 177.8 59.055 180)
     (effects (font (size 1.27 1.27)) (justify right bottom))
   )
-  (label "MISO" (at 167.513 85.09 90)
-    (effects (font (size 1.27 1.27)) (justify left bottom))
-  )
-  (label "MOSI" (at 198.755 58.42 0)
-    (effects (font (size 1.27 1.27)) (justify left bottom))
-  )
-  (label "MISO" (at 177.8 55.88 180)
+  (label "MISO_JTAG" (at 167.513 85.09 90)
+    (effects (font (size 1.27 1.27)) (justify left bottom))
+  )
+  (label "MOSI_JTAG" (at 198.755 58.42 0)
+    (effects (font (size 1.27 1.27)) (justify left bottom))
+  )
+  (label "MISO_JTAG" (at 177.8 55.88 180)
     (effects (font (size 1.27 1.27)) (justify right bottom))
   )
-  (label "MOSI" (at 164.338 85.09 90)
-    (effects (font (size 1.27 1.27)) (justify left bottom))
-  )
-  (label "SCK" (at 161.163 85.09 90)
-    (effects (font (size 1.27 1.27)) (justify left bottom))
-  )
-  (hierarchical_label "Relay_1" (shape input) (at 145.796 102.87 0)
+  (label "MOSI_JTAG" (at 164.338 85.09 90)
+    (effects (font (size 1.27 1.27)) (justify left bottom))
+  )
+  (label "SCK_JTAG" (at 161.163 85.09 90)
+    (effects (font (size 1.27 1.27)) (justify left bottom))
+  )
+  (hierarchical_label "igniter2" (shape input) (at 145.796 102.87 0)
     (effects (font (size 1.27 1.27)) (justify left))
   )
@@
     (effects (font (size 1.27 1.27)) (justify left))
   )
-  (hierarchical_label "Relay_2" (shape input) (at 145.923 100.33 0)
+  (hierarchical_label "igniter3" (shape input) (at 145.923 100.33 0)
     (effects (font (size 1.27 1.27)) (justify left))
   )
@@
   )
   (hierarchical_label "SD_CS" (shape input) (at 144.399 95.25 0)
+    (effects (font (size 1.27 1.27)) (justify left))
+  )
+  (hierarchical_label "SD_CD" (shape input) (at 143.637 153.67 0)
     (effects (font (size 1.27 1.27)) (justify left))
   )
@@
     (effects (font (size 1.27 1.27)) (justify left))
   )
-  (hierarchical_label "IGNITION" (shape input) (at 145.796 105.41 0)
-    (effects (font (size 1.27 1.27)) (justify left))
-  )
+  (hierarchical_label "igniter1" (shape input) (at 145.796 105.41 0)
+    (effects (font (size 1.27 1.27)) (justify left))
+  )
