File: MainRework/Recovery_DoubleStage.kicad_pcb (KiCad board)
At the start: 4 copper layers, 100.6 x 76.7 mm, 68 parts, among them IC1 ATMEGA2560-16AU, IC2 AP2210N-3.3TRG1, IC3 MMC5983MA, IC4 NEO-6M-0, IC5 BMP388, IC6 MPU-6050, J1 ICSP, J2 Conn_02x10_Counter_Clockwise, J3 Conn_Coaxial, J4 Conn_Coaxial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

Commit message: reworking
Parts:
- moved J3 10.3 mm to (118.3, 79.0)
- moved J4 9.55 mm to (117.5, 25.7)
Changed lines of the file:
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@@
   )
   (footprint "Footprint:RF_Solutions_Ltd.-CON-SMA-EDGE-S-MFG" (layer "F.Cu")
-    (at 107.917 78.9432 -90)
+    (at 118.258 79.0448 -90)
     (property "Sheetfile" "Recovery_DoubleStage.kicad_sch")
     (property "Sheetname" "")
@@
   )
   (footprint "Footprint:RF_Solutions_Ltd.-CON-SMA-EDGE-S-MFG" (layer "F.Cu")
-    (at 107.95 25.654 -90)
-    (property "Sheetfile" "Recovery_DoubleStage.kicad_sch")
-    (property "Sheetname" "")
+    (at 117.496 25.654 -90)
+    (property "Sheetfile" "Recovery_DoubleStage.kicad_sch")
+    (property "Sheetname" "")
