File: MainRework/mpu mmc.kicad_sch (KiCad schematic)
At the start: 55 parts, among them IC2 AP2210N-3.3TRG1, IC3 MMC5983MA, IC4 NEO-6M-0, IC5 BMP388, IC6 MPU-6050, J2 Conn_02x10_Counter_Clockwise, J3 Conn_Coaxial, J4 Conn_Coaxial, J5 MEM2075-00-140-01-A, J6 JSTXH-1x02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

Commit message: reworking
Parts:
- removed H1, H2, H3, H4: MountingHole, MountingHole:MountingHole_2.1mm, symbol Mechanical:MountingHole
- removed J6: JSTXH-1x02, Connector_JST:JST_XH_B2B-XH-AM_1x02_P2.50mm_Vertical, symbol XT60PW-M:XT60PW-M
- added J6: Conn_01x02_Female, symbol Connector:Conn_01x02_Female
- added R5: 2.7k, Resistor_SMD:R_0603_1608Metric, symbol Device:R
- added TP7: MISO, TestPoint:TestPoint_Pad_D1.0mm, symbol Connector:TestPoint
- added TP8: MOSI, TestPoint:TestPoint_Pad_D1.0mm, symbol Connector:TestPoint
- added TP9: SCK, TestPoint:TestPoint_Pad_D1.0mm, symbol Connector:TestPoint
- BZ1: footprint custom:TE054003 -> (none)
Connections:
- net +3V3: no longer C20.2, C22.1, IC2.2 (VOUT), IC3.13 (VDDIO), IC3.2 (VDD), IC3.4 (SPI_CS)
- net +5V: now also BZ1.1 (-), U1. (VOUT); no longer BZ1.2 (+), U1.3 (VOUT)
- net +BATT: now also U1. (VOUT), J6.1 (Pin_1); no longer U1.1 (VIN)
- net GND: now also U1. (VOUT), J6.2 (Pin_2); no longer C7.1, IC6.18 (GND), U1.2 (GND)
- net MISO: now also TP7.1
- net MOSI: now also TP8.1
- net SCK: now also IC3.1 (SCL/SPI_SCK), TP9.1
- net SCL: no longer IC3.1 (SCL/SPI_SCK)
- net SDA: no longer IC3.16 (SDA/SPI_SDI)
- net at D2.1 (A), Q1.3 (D): now also BZ1.2 (+); no longer BZ1.3 (+)
- net ANT_LORA: no longer names the net of J4.1 (In), U2.9 (ANT)
- net ANT_NEO: no longer names the net of IC4.11 (RF_IN), J3.1 (In), L1.2
- new net: C22.1, IC3.13 (VDDIO), IC3.2 (VDD), IC3.4 (SPI_CS), R5.1
- new net: IC3.16 (SDA/SPI_SDI), R5.2
- new net: C20.2, IC2.2 (VOUT)
- new net: C7.1, IC6.18 (GND)
- no-connect marks 41 -> 42
